File: Rev A.sch (EAGLE design)
At the start: 0 parts

Commit message: Finished the schematic
Parts:
- added C1, C1001: 100pF, rcl:C-EU050-050X075
- added C1002, C2: 4.7uF, rcl:C-EU225-113X268
- added C1003, C3: 4.7uF, rcl:CPOL-EUE2-5
- added C201, C202: 0.1uF, rcl:C-EU025-025X050
- added C203, C204: 1000uF, rcl:CPOL-EUE5-10.5
- added C301, C302: 10uF, rcl:CPOL-EUE2.5-6
- added D1, D1001, D2, D3, D4, D5, D6, D7: 1N4148DO35-7, diode:1N4148DO35-7
- added D301, D302: 6.2V, diode:ZENER-DIODEDO34-7
- added F1, F2: 2A, fuse:SH22,5
- added IC301: LM339N, linear:LM339N
- added L_CLIP, R_CLIP: (no value), adafruit:LED5MM
- added L_IN, L_OUT1, L_OUT2, PWR+, PWR-, R_IN, R_OUT1, R_OUT2: (no value), adafruit:JST_2PIN-THM
- added ON+, ON-: (no value), led:LEDSQR2X5
- added Q1, Q10, Q1002, Q11, Q2, Q9: 2N3906, transistor-pnp:2N3906
- added Q1001, Q12, Q13, Q14, Q3, Q4, Q5, Q8: 2N3904, transistor-npn:2N3904
- added Q15, Q6: TIP41C, transistor-power:TIP41C
- added Q16, Q7: TIP42C, transistor-power:TIP42C
- added R1, R10, R16, R301, R302, R303, R304, R8: 10kΩ, rcl:R-EU_0207/10
- added R11, R2: 8.2kΩ, rcl:R-EU_0207/10
- added R12, R201, R202, R3, R313, R314: 2.2kΩ, rcl:R-EU_0207/10
- added R13, R15, R305, R306, R4, R7: 1kΩ, rcl:R-EU_0207/10
- added R14, R18, R5, R6: 0.33, rcl:R-EU_0414/15
- added R17, R9: 180kΩ, rcl:R-EU_0207/10
- added R307, R308, R310, R312: 100kΩ, rcl:R-EU_0207/10
- added R309, R311: 56kΩ, rcl:R-EU_0207/10
- added VR301, VR302: 10kΩ, bourns:3362U
Connections:
- new net GND: C203.-, C204.+, D301.A, D302.A, L_IN.2, L_OUT1.2, L_OUT2.2, PWR+.2, PWR-.1, R1.1, R10.1, R16.1, R201.1, R202.1, R303.2, R304.2, R8.1, R_IN.2, R_OUT1.2, R_OUT2.2, VR301.3, VR302.3
- new net L_OUT: D4.A, D7.C, L_OUT1.1, L_OUT2.1, R14.1, R17.2, R18.2, R302.1
- new net N$1: D2.A, Q1001.B, R3.1
- new net N$10: IC301A.+IN, VR301.2
- new net N$11: D301.C, R305.1, VR301.1
- new net N$12: C301.+, IC301A.OUT, IC301B.-IN, R307.1
- new net N$13: IC301B.+IN, R309.1, R310.2
- new net N$14: IC301B.OUT, R_CLIP.C
- new net N$15: R313.1, R_CLIP.A
- new net N$16: IC301C.-IN, R302.2, R304.1
- new net N$17: IC301C.+IN, VR302.2
- new net N$18: D302.C, R306.1, VR302.1
- new net N$19: C302.+, IC301C.OUT, IC301D.-IN, R308.1
- new net N$2: Q1.E, Q2.E, R2.1
- new net N$20: IC301D.+IN, R311.1, R312.2
- new net N$21: IC301D.OUT, L_CLIP.C
- new net N$22: ON+.C, R201.2
- new net N$23: L_CLIP.A, R314.1
- new net N$24: D1.A, D2.C
- new net N$25: C2.2, C3.-, Q10.B, R10.2
- new net N$26: Q1001.C, Q7.B, R4.1
- new net N$27: Q1002.C, Q6.B, R7.2
- new net N$28: Q1002.E, Q6.C, R6.1
- new net N$29: Q1001.E, Q7.C, R5.2
- new net N$3: Q2.C, Q3.B, Q3.C, Q4.B
- new net N$30: C2.1, C3.+, L_IN.1
- new net N$31: C1001.2, D1.C, Q1002.B, Q5.C
- new net N$32: Q2.B, R8.2, R9.1
- new net N$33: Q10.E, Q11.E, R11.1
- new net N$34: C1.1, Q10.C, Q13.C, Q14.B
- new net N$35: D5.A, D6.C
- new net N$36: D6.A, Q8.B, R12.1
- new net N$37: Q16.B, Q8.C, R13.1
- new net N$38: Q16.C, Q8.E, R14.2
- new net N$39: Q15.B, Q9.C, R15.2
- new net N$4: Q11.C, Q12.B, Q12.C, Q13.B
- new net N$40: Q15.C, Q9.E, R18.1
- new net N$41: C1.2, D5.C, Q14.C, Q9.B
- new net N$42: Q11.B, R16.2, R17.1
- new net N$43: F1.1, PWR+.1
- new net N$44: F2.2, PWR-.2
- new net N$5: C1002.2, C1003.-, Q1.B, R1.2
- new net N$6: C1002.1, C1003.+, R_IN.1
- new net N$7: ON-.A, R202.2
- new net N$8: C1001.1, Q1.C, Q4.C, Q5.B
- new net N$9: IC301A.-IN, R301.2, R303.1
- new net R_OUT: D1001.A, D3.C, R301.1, R5.1, R6.2, R9.2, R_OUT1.1, R_OUT2.1
- new net V+: C201.1, C202.1, C203.+, D1001.C, D4.C, F1.2, IC301P.V+, ON+.A, Q16.E, Q7.E, R11.2, R12.2, R13.2, R2.2, R3.2, R305.2, R306.2, R307.2, R308.2, R309.2, R311.2, R313.2, R314.2, R4.2
- new net V-: C201.2, C202.2, C204.-, C301.-, C302.-, D3.A, D7.A, F2.1, IC301P.GND, ON-.C, Q12.E, Q13.E, Q14.E, Q15.E, Q3.E, Q4.E, Q5.E, Q6.E, R15.1, R310.1, R312.1, R7.1
