File: Rev A.sch (EAGLE design)
At the start: 70 parts, among them Q101 2N3906, Q102 2N3906, Q103 2N3904, Q104 2N3904, Q105 2N3904, Q106 2N3904, Q107 2N3906, Q108 2N3906, Q109 2N3904, Q110 2N3904, Q111 2N3904, Q112 2N3906, Q113 2N3904, Q114 2N3906, Q115 TIP42C, Q116 TIP41C, Q117 TIP42C, Q118 TIP41C

Commit message: Final changes
Parts:
- added H201, H202, H203, H204: MOUNT-HOLE3.0, holes:MOUNT-HOLE3.0
- renumbered C203 to C201, C204 to C202, L_OUT1 to L_OUT101, L_OUT2 to L_OUT102, R_OUT1 to R_OUT101, R_OUT2 to R_OUT102
Connections:
- net N$43: now also SWT+2.1, SWT+2.2; no longer SWT+1.1, SWT+1.2
- net N$47: now also SWT+1.1, SWT+1.2; no longer SWT+2.1, SWT+2.2
Other:
- moved on the sheet: SWT+1, SWT+2
Changed lines of the file:
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@@
 <part name="C101" library="rcl" deviceset="C-EU" device="225-113X268" value="4.7uF"/>
 <part name="C102" library="rcl" deviceset="CPOL-EU" device="E2-5" value="4.7uF"/>
-<part name="C204" library="rcl" deviceset="CPOL-EU" device="E5-10.5" value="1000uF"/>
-<part name="C203" library="rcl" deviceset="CPOL-EU" device="E5-10.5" value="1000uF"/>
+<part name="C202" library="rcl" deviceset="CPOL-EU" device="E5-10.5" value="1000uF"/>
+<part name="C201" library="rcl" deviceset="CPOL-EU" device="E5-10.5" value="1000uF"/>
 <part name="Q101" library="transistor-pnp" deviceset="2N3906" device=""/>
 <part name="Q107" library="transistor-pnp" deviceset="2N3906" device=""/>
@@
 <part name="PWR-1" library="adafruit" deviceset="JST_2PIN" device="-THM"/>
 <part name="PWR-2" library="adafruit" deviceset="JST_2PIN" device="-THM"/>
-<part name="R_OUT1" library="adafruit" deviceset="JST_2PIN" device="-THM"/>
-<part name="R_OUT2" library="adafruit" deviceset="JST_2PIN" device="-THM"/>
-<part name="L_OUT1" library="adafruit" deviceset="JST_2PIN" device="-THM"/>
-<part name="L_OUT2" library="adafruit" deviceset="JST_2PIN" device="-THM"/>
+<part name="R_OUT101" library="adafruit" deviceset="JST_2PIN" device="-THM"/>
+<part name="R_OUT102" library="adafruit" deviceset="JST_2PIN" device="-THM"/>
+<part name="L_OUT101" library="adafruit" deviceset="JST_2PIN" device="-THM"/>
+<part name="L_OUT102" library="adafruit" deviceset="JST_2PIN" device="-THM"/>
 <part name="R_IN" library="adafruit" deviceset="JST_2PIN" device="-THM"/>
 <part name="L_IN" library="adafruit" deviceset="JST_2PIN" device="-THM"/>
+<part name="SWT+1" library="adafruit" deviceset="JST_2PIN" device="-THM"/>
 <part name="SWT+2" library="adafruit" deviceset="JST_2PIN" device="-THM"/>
-<part name="SWT+1" library="adafruit" deviceset="JST_2PIN" device="-THM"/>
 <part name="SWT-1" library="adafruit" deviceset="JST_2PIN" device="-THM"/>
 <part name="SWT-2" library="adafruit" deviceset="JST_2PIN" device="-THM"/>
 <part name="SUPPLY10" library="supply2" deviceset="V-" device=""/>
 <part name="LED" library="adafruit" deviceset="JST_2PIN" device="-THM"/>
+<part name="H201" library="holes" deviceset="MOUNT-HOLE" device="3.0"/>
+<part name="H202" library="holes" deviceset="MOUNT-HOLE" device="3.0"/>
+<part name="H203" library="holes" deviceset="MOUNT-HOLE" device="3.0"/>
+<part name="H204" library="holes" deviceset="MOUNT-HOLE" device="3.0"/>
 </parts>
 <sheets>
@@
 <attribute name="NAME" x="52.8574" y="-17.78" size="1.778" layer="95" rot="R90"/>
 </instance>
-<instance part="R_OUT1" gate="G$1" x="78.74" y="109.22" rot="MR180"/>
-<instance part="R_OUT2" gate="G$1" x="78.74" y="99.06" rot="MR180"/>
-<instance part="L_OUT1" gate="G$1" x="78.74" y="-10.16" rot="MR180"/>
-<instance part="L_OUT2" gate="G$1" x="78.74" y="-20.32" rot="MR180"/>
+<instance part="R_OUT101" gate="G$1" x="78.74" y="109.22" rot="MR180"/>
+<instance part="R_OUT102" gate="G$1" x="78.74" y="99.06" rot="MR180"/>
+<instance part="L_OUT101" gate="G$1" x="78.74" y="-10.16" rot="MR180"/>
+<instance part="L_OUT102" gate="G$1" x="78.74" y="-20.32" rot="MR180"/>
 <instance part="R_IN" gate="G$1" x="-83.82" y="106.68" rot="R180"/>
 <instance part="L_IN" gate="G$1" x="-83.82" y="-12.7" rot="R180"/>
@@
 <wire x1="68.58" y1="96.52" x2="68.58" y2="88.9" width="0.1524" layer="91"/>
 <pinref part="GND7" gate="1" pin="GND"/>
-<pinref part="R_OUT2" gate="G$1" pin="1"/>
-<pinref part="R_OUT2" gate="G$1" pin="2"/>
+<pinref part="R_OUT102" gate="G$1" pin="1"/>
+<pinref part="R_OUT102" gate="G$1" pin="2"/>
 <wire x1="68.58" y1="99.06" x2="76.2" y2="99.06" width="0.1524" layer="91"/>
 <wire x1="68.58" y1="99.06" x2="68.58" y2="96.52" width="0.1524" layer="91"/>
@@
 <wire x1="68.58" y1="-22.86" x2="68.58" y2="-30.48" width="0.1524" layer="91"/>
 <pinref part="GND11" gate="1" pin="GND"/>
-<pinref part="L_OUT2" gate="G$1" pin="1"/>
-<pinref part="L_OUT2" gate="G$1" pin="2"/>
+<pinref part="L_OUT102" gate="G$1" pin="1"/>
+<pinref part="L_OUT102" gate="G$1" pin="2"/>
 <wire x1="68.58" y1="-20.32" x2="76.2" y2="-20.32" width="0.1524" layer="91"/>
 <wire x1="68.58" y1="-20.32" x2="68.58" y2="-22.86" width="0.1524" layer="91"/>
@@
 <junction x="53.34" y="106.68"/>
 <label x="55.88" y="106.68" size="1.778" layer="95"/>
-<pinref part="R_OUT1" gate="G$1" pin="2"/>
-<pinref part="R_OUT1" gate="G$1" pin="1"/>
+<pinref part="R_OUT101" gate="G$1" pin="2"/>
+<pinref part="R_OUT101" gate="G$1" pin="1"/>
 <wire x1="76.2" y1="106.68" x2="68.58" y2="106.68" width="0.1524" layer="91"/>
 <junction x="68.58" y="106.68"/>
@@
 <junction x="53.34" y="-12.7"/>
 <label x="55.88" y="-12.7" size="1.778" layer="95"/>
-<pinref part="L_OUT1" gate="G$1" pin="2"/>
-<pinref part="L_OUT1" gate="G$1" pin="1"/>
+<pinref part="L_OUT101" gate="G$1" pin="2"/>
+<pinref part="L_OUT101" gate="G$1" pin="1"/>
 <wire x1="76.2" y1="-12.7" x2="68.58" y2="-12.7" width="0.1524" layer="91"/>
 <junction x="68.58" y="-12.7"/>
@@
 <instance part="GND14" gate="1" x="25.4" y="121.92" rot="R180"/>
 <instance part="SUPPLY12" gate="1" x="25.4" y="50.8"/>
-<instance part="C204" gate="G$1" x="60.96" y="76.2"/>
-<instance part="C203" gate="G$1" x="50.8" y="73.66" rot="R180"/>
+<instance part="C202" gate="G$1" x="60.96" y="76.2"/>
+<instance part="C201" gate="G$1" x="50.8" y="73.66" rot="R180"/>
 <instance part="F201" gate="1" x="-2.54" y="109.22" rot="R90"/>
 <instance part="F202" gate="1" x="25.4" y="63.5" rot="R90"/>
@@
 <instance part="PWR-1" gate="G$1" x="35.56" y="114.3" rot="MR180"/>
 <instance part="PWR-2" gate="G$1" x="35.56" y="101.6" rot="MR180"/>
-<instance part="SWT+2" gate="G$1" x="10.16" y="101.6" rot="MR180"/>
-<instance part="SWT+1" gate="G$1" x="10.16" y="88.9" rot="MR180"/>
+<instance part="SWT+1" gate="G$1" x="10.16" y="101.6" rot="MR180"/>
+<instance part="SWT+2" gate="G$1" x="10.16" y="88.9" rot="MR180"/>
 <instance part="SWT-1" gate="G$1" x="35.56" y="88.9" rot="MR180"/>
 <instance part="SWT-2" gate="G$1" x="35.56" y="76.2" rot="MR180"/>
 <instance part="SUPPLY10" gate="1" x="71.12" y="55.88"/>
 <instance part="LED" gate="G$1" x="76.2" y="83.82" rot="MR180"/>
+<instance part="H201" gate="G$1" x="50.8" y="124.46"/>
+<instance part="H202" gate="G$1" x="50.8" y="116.84"/>
+<instance part="H203" gate="G$1" x="50.8" y="109.22"/>
+<instance part="H204" gate="G$1" x="50.8" y="101.6"/>
 </instances>
 <busses>
@@
 <wire x1="60.96" y1="71.12" x2="60.96" y2="58.42" width="0.1524" layer="91"/>
 <pinref part="GND13" gate="1" pin="GND"/>
-<pinref part="C204" gate="G$1" pin="-"/>
+<pinref part="C202" gate="G$1" pin="-"/>
 </segment>
 <segment>
 <wire x1="50.8" y1="71.12" x2="50.8" y2="58.42" width="0.1524" layer="91"/>
 <pinref part="GND6" gate="1" pin="GND"/>
-<pinref part="C203" gate="G$1" pin="+"/>
+<pinref part="C201" gate="G$1" pin="+"/>
 </segment>
 <segment>
@@
 <wire x1="50.8" y1="78.74" x2="50.8" y2="91.44" width="0.1524" layer="91"/>
 <pinref part="SUPPLY7" gate="1" pin="V-"/>
-<pinref part="C203" gate="G$1" pin="-"/>
+<pinref part="C201" gate="G$1" pin="-"/>
 </segment>
 <segment>
@@
 <wire x1="60.96" y1="78.74" x2="60.96" y2="91.44" width="0.1524" layer="91"/>
 <pinref part="SUPPLY8" gate="1" pin="V+"/>
-<pinref part="C204" gate="G$1" pin="+"/>
+<pinref part="C202" gate="G$1" pin="+"/>
 </segment>
 <segment>
@@
 <wire x1="0" y1="76.2" x2="7.62" y2="76.2" width="0.1524" layer="91"/>
 <pinref part="PWR+1" gate="G$1" pin="2"/>
-<pinref part="SWT+1" gate="G$1" pin="2"/>
+<pinref part="SWT+2" gate="G$1" pin="2"/>
 <wire x1="7.62" y1="88.9" x2="0" y2="88.9" width="0.1524" layer="91"/>
 <wire x1="0" y1="88.9" x2="0" y2="86.36" width="0.1524" layer="91"/>
-<pinref part="SWT+1" gate="G$1" pin="1"/>
+<pinref part="SWT+2" gate="G$1" pin="1"/>
 <wire x1="0" y1="86.36" x2="0" y2="76.2" width="0.1524" layer="91"/>
 <wire x1="7.62" y1="86.36" x2="0" y2="86.36" width="0.1524" layer="91"/>
@@
 <net name="N$47" class="0">
 <segment>
-<pinref part="SWT+2" gate="G$1" pin="2"/>
-<pinref part="SWT+2" gate="G$1" pin="1"/>
+<pinref part="SWT+1" gate="G$1" pin="2"/>
+<pinref part="SWT+1" gate="G$1" pin="1"/>
 <wire x1="-2.54" y1="99.06" x2="7.62" y2="99.06" width="0.1524" layer="91"/>
 <wire x1="-2.54" y1="99.06" x2="-2.54" y2="101.6" width="0.1524" layer="91"/>
